File: schematic/quadcopter/quadcopter.sch (KiCad schematic (older format))
At the start: 1 part

Commit message: Update quadcopter schematic
Parts:
- removed U??: weact_stm32f411ceu6, symbol quadcopter_symbol:weact_stm32f411ceu6
- added U1: WEACT_STM32F411CEU6, symbol quadcopter_symbol:WEACT_STM32F411CEU6
- added U10, U11, U12, U13: iFlight_XING_E_2207, symbol quadcopter_symbol:iFlight_XING_E_2207
- added U2: SPARKRUN_ICM-20948, symbol quadcopter_symbol:SPARKRUN_ICM-20948
- added U3: LIPO_Battery_4CELL, symbol quadcopter_symbol:LIPO_Battery_4CELL
- added U4: FS-A8S, symbol quadcopter_symbol:FS-A8S
- added U5: MATEK_PDB-XT60, symbol quadcopter_symbol:MATEK_PDB-XT60
- added U6, U7, U8, U9: HAKRC_35A_ESC, symbol quadcopter_symbol:HAKRC_35A_ESC
Connections:
- net labels added: +5V, CS, MISO, MOSI, SCLK, TIM2_CH3, TIM2_CH4, TIM5_CH1, TIM5_CH2, USART1_RX, VCC
- wire segments 6 -> 62
Other:
- note added: "IMU (ICM-20948)"
- note added: "MCU"
- note added: "Motor"
- note added: "Motor 1"
- note added: "Motor 2"
- note added: "Motor 3"
- note added: "Motor 4"
- note added: "PDB"
- note added: "RC Receiver (FS-A8S)"
